Commit message: Working on simulation

File: franka_description/robots/hand.xacro (robot description, xacro)
@@ -52,4 +52,14 @@
         </geometry>
       </collision>
+      <collision>
+        <geometry>
+          <mesh filename="package://franka_description/meshes/collision/hand.stl"/>
+        </geometry>
+      </collision>
+      <inertial>
+        <origin xyz="0 0 0" rpy="0 0 0"/>
+        <mass value="0.68"/>
+        <inertia ixx="0.1" ixy="0.0" ixz="0.0" iyy="0.1" iyz="0.0" izz="0.1"/>
+      </inertial>
     </link>
     <link name="${ns}_leftfinger">
@@ -59,4 +69,14 @@
         </geometry>
       </visual>
+      <collision>
+        <geometry>
+          <mesh filename="package://franka_description/meshes/collision/finger.stl"/>
+        </geometry>
+      </collision>
+      <inertial>
+        <origin xyz="0 0 0" rpy="0 0 0"/>
+        <mass value="0.01"/>
+        <inertia ixx="0.1" ixy="0.0" ixz="0.0" iyy="0.1" iyz="0.0" izz="0.1"/>
+      </inertial>
     </link>
     <link name="${ns}_rightfinger">
@@ -67,4 +87,14 @@
         </geometry>
       </visual>
+      <collision>
+        <geometry>
+          <mesh filename="package://franka_description/meshes/collision/finger.stl"/>
+        </geometry>
+      </collision>
+      <inertial>
+        <origin xyz="0 0 0" rpy="0 0 0"/>
+        <mass value="0.01"/>
+        <inertia ixx="0.1" ixy="0.0" ixz="0.0" iyy="0.1" iyz="0.0" izz="0.1"/>
+      </inertial>
    </link>
     <joint name="${ns}_finger_joint1" type="prismatic">

File: franka_description/robots/panda_arm.xacro (robot description, xacro)
@@ -11,4 +11,12 @@
       </joint>
     </xacro:unless>
+    <xacro:property name="joint_damping" value="1.0"/>
+    <link name="world" />
+    <joint name="robot_to_world" type="fixed">
+      <parent link="world" />
+      <child link="${arm_id}_link0" />
+      <origin xyz="0.0 0.0 0.0" rpy="0.0 0.0 0.0" />
+      <dynamics damping="${joint_damping}"/>
+    </joint>
     <link name="${arm_id}_link0">
       <visual>
@@ -35,4 +43,9 @@
         </geometry>
       </collision>
+      <inertial>
+        <origin xyz="0 0 0" rpy="0 0 0"/>
+        <mass value="3.06"/>
+        <inertia ixx="0.3" ixy="0.0" ixz="0.0" iyy="0.3" iyz="0.0" izz="0.3"/>
+      </inertial>
     </link>
     <link name="${arm_id}_link1">
@@ -60,4 +73,9 @@
         </geometry>
       </collision>
+      <inertial>
+        <origin xyz="0 0 0" rpy="0 0 0"/>
+        <mass value="2.34"/>
+        <inertia ixx="0.3" ixy="0.0" ixz="0.0" iyy="0.3" iyz="0.0" izz="0.3"/>
+      </inertial>
     </link>
     <joint name="${arm_id}_joint1" type="revolute">
@@ -68,5 +86,6 @@
       <axis xyz="0 0 1"/>
       <limit effort="87" lower="-2.8973" upper="2.8973" velocity="2.1750"/>
-    </joint>
+      <dynamics damping="${joint_damping}"/>
+   </joint>
     <link name="${arm_id}_link2">
       <visual>
@@ -93,4 +112,9 @@
         </geometry>
       </collision>
+      <inertial>
+        <origin xyz="0 0 0" rpy="0 0 0"/>
+        <mass value="2.36"/>
+        <inertia ixx="0.3" ixy="0.0" ixz="0.0" iyy="0.3" iyz="0.0" izz="0.3"/>
+      </inertial>
     </link>
     <joint name="${arm_id}_joint2" type="revolute">
@@ -101,4 +125,5 @@
       <axis xyz="0 0 1"/>
       <limit effort="87" lower="-1.7628" upper="1.7628" velocity="2.1750"/>
+      <dynamics damping="${joint_damping}"/>
     </joint>
     <link name="${arm_id}_link3">
@@ -126,4 +151,9 @@
         </geometry>
       </collision>
+      <inertial>
+        <origin xyz="0 0 0" rpy="0 0 0"/>
+        <mass value="2.38"/>
+        <inertia ixx="0.3" ixy="0.0" ixz="0.0" iyy="0.3" iyz="0.0" izz="0.3"/>
+      </inertial>
     </link>
     <joint name="${arm_id}_joint3" type="revolute">
@@ -134,4 +164,5 @@
       <axis xyz="0 0 1"/>
       <limit effort="87" lower="-2.8973" upper="2.8973" velocity="2.1750"/>
+      <dynamics damping="${joint_damping}"/>
     </joint>
     <link name="${arm_id}_link4">
@@ -159,4 +190,9 @@
         </geometry>
       </collision>
+      <inertial>
+        <origin xyz="0 0 0" rpy="0 0 0"/>
+        <mass value="2.43"/>
+        <inertia ixx="0.3" ixy="0.0" ixz="0.0" iyy="0.3" iyz="0.0" izz="0.3"/>
+      </inertial>
     </link>
     <joint name="${arm_id}_joint4" type="revolute">
@@ -167,4 +203,5 @@
       <axis xyz="0 0 1"/>
       <limit effort="87" lower="-3.0718" upper="-0.0698" velocity="2.1750"/>
+      <dynamics damping="${joint_damping}"/>
     </joint>
     <link name="${arm_id}_link5">
@@ -210,4 +247,9 @@
         </geometry>
       </collision>
+      <inertial>
+        <origin xyz="0 0 0" rpy="0 0 0"/>
+        <mass value="3.5"/>
+        <inertia ixx="0.3" ixy="0.0" ixz="0.0" iyy="0.3" iyz="0.0" izz="0.3"/>
+      </inertial>
     </link>
     <joint name="${arm_id}_joint5" type="revolute">
@@ -218,4 +260,5 @@
       <axis xyz="0 0 1"/>
       <limit effort="12" lower="-2.8973" upper="2.8973" velocity="2.6100"/>
+      <dynamics damping="${joint_damping}"/>
     </joint>
     <link name="${arm_id}_link6">
@@ -243,4 +286,9 @@
         </geometry>
       </collision>
+      <inertial>
+        <origin xyz="0 0 0" rpy="0 0 0"/>
+        <mass value="1.47"/>
+        <inertia ixx="0.3" ixy="0.0" ixz="0.0" iyy="0.3" iyz="0.0" izz="0.3"/>
+      </inertial>
     </link>
     <joint name="${arm_id}_joint6" type="revolute">
@@ -251,4 +299,5 @@
       <axis xyz="0 0 1"/>
       <limit effort="12" lower="-0.0175" upper="3.7525" velocity="2.6100"/>
+      <dynamics damping="${joint_damping}"/>
     </joint>
     <link name="${arm_id}_link7">
@@ -276,4 +325,9 @@
         </geometry>
       </collision>
+      <inertial>
+        <origin xyz="0 0 0" rpy="0 0 0"/>
+        <mass value="0.45"/>
+        <inertia ixx="0.3" ixy="0.0" ixz="0.0" iyy="0.3" iyz="0.0" izz="0.3"/>
+      </inertial>
     </link>
     <joint name="${arm_id}_joint7" type="revolute">
@@ -284,4 +338,5 @@
       <axis xyz="0 0 1"/>
       <limit effort="12" lower="-2.8973" upper="2.8973" velocity="2.6100"/>
+      <dynamics damping="${joint_damping}"/>
     </joint>
     <link name="${arm_id}_link8">
@@ -304,4 +359,9 @@
         </geometry>
       </collision>
+      <inertial>
+        <origin xyz="0 0 0" rpy="0 0 0"/>
+        <mass value="0.0"/>
+        <inertia ixx="0.3" ixy="0.0" ixz="0.0" iyy="0.3" iyz="0.0" izz="0.3"/>
+      </inertial>
     </link>
     <joint name="${arm_id}_joint8" type="fixed">

File: franka_description/robots/panda_arm_hand.urdf.xacro (robot description, xacro)
@@ -1,7 +1,12 @@
 <?xml version="1.0" encoding="utf-8"?>
 <robot xmlns:xacro="http://www.ros.org/wiki/xacro" name="panda">
+  <xacro:arg name="robot_name" default="panda"/>
   <xacro:include filename="$(find franka_description)/robots/panda_arm.xacro"/>
   <xacro:include filename="$(find franka_description)/robots/hand.xacro"/>
+  <xacro:include filename="$(find franka_description)/robots/panda.gazebo.xacro"/>
+  <xacro:include filename="$(find franka_description)/robots/panda.transmission.xacro"/>
   <xacro:panda_arm safety_distance="0.03"/>
   <xacro:hand ns="panda" rpy="0 0 ${-pi/4}" connected_to="panda_link8" safety_distance="0.03"/>
+  <xacro:panda_gazebo robot_name="$(arg robot_name)" />
+  <xacro:panda_transmission robot_name="$(arg robot_name)" />
 </robot>

Commit message: Not working version

File: franka_description/robots/hand.xacro (robot description, xacro)
@@ -52,4 +52,16 @@
         </geometry>
       </collision>
+      <collision>
+        <geometry>
+          <mesh filename="package://franka_description/meshes/collision/hand.stl"/>
+        </geometry>
+      </collision>
+      <!-- for simulation -->
+      <inertial>
+        <origin xyz="0 0 0" rpy="0 0 0" />
+        <mass value="0.68" />
+        <inertia ixx="0.1" ixy="0.0" ixz="0.0" iyy="0.1" iyz="0.0" izz="0.1" />
+      </inertial>
+      <!-- end for simulation -->
     </link>
     <link name="${ns}_leftfinger">
@@ -59,4 +71,16 @@
         </geometry>
       </visual>
+      <collision>
+        <geometry>
+          <mesh filename="package://franka_description/meshes/collision/finger.stl"/>
+        </geometry>
+      </collision>
+      <!-- for simulation -->
+      <inertial>
+        <origin xyz="0 0 0" rpy="0 0 0" />
+        <mass value="0.01" />
+        <inertia ixx="0.1" ixy="0.0" ixz="0.0" iyy="0.1" iyz="0.0" izz="0.1" />
+      </inertial>
+      <!-- end for simulation -->
     </link>
     <link name="${ns}_rightfinger">
@@ -67,4 +91,17 @@
         </geometry>
       </visual>
+      <collision>
+        <origin xyz="0 0 0" rpy="0 0 ${pi}"/>
+        <geometry>
+          <mesh filename="package://franka_description/meshes/collision/finger.stl"/>
+        </geometry>
+      </collision>
+      <!-- for simulation -->
+      <inertial>
+        <origin xyz="0 0 0" rpy="0 0 0" />
+        <mass value="0.01" />
+        <inertia ixx="0.1" ixy="0.0" ixz="0.0" iyy="0.1" iyz="0.0" izz="0.1" />
+      </inertial>
+      <!-- end for simulation -->
    </link>
     <joint name="${ns}_finger_joint1" type="prismatic">
@@ -81,5 +118,4 @@
       <axis xyz="0 -1 0"/>
       <limit effort="20" lower="0.0" upper="0.04" velocity="0.2"/>
-      <mimic joint="${ns}_finger_joint1" />
     </joint>
   </xacro:macro>

File: franka_description/robots/panda_arm.urdf.xacro (robot description, xacro)
@@ -2,4 +2,13 @@
 <robot xmlns:xacro="http://www.ros.org/wiki/xacro" name="panda">
   <xacro:include filename="$(find franka_description)/robots/panda_arm.xacro" />
+  <!-- for simulation -->
+  <xacro:include filename="$(find franka_description)/robots/panda.gazebo.xacro"/>
+  <xacro:include filename="panda.transmission.xacro"/>
+  <!-- end for simulation -->
   <xacro:panda_arm safety_distance="0.03"/>
+  <!-- for simulation -->
+  <xacro:arg name="robot_name" default="panda"/>
+  <xacro:panda_gazebo robot_name="$(arg robot_name)" />
+  <xacro:panda_transmission robot_name="$(arg robot_name)" load_hand="false" />
+  <!-- end for simulation -->
 </robot>

File: franka_description/robots/panda_arm.xacro (robot description, xacro)
@@ -11,4 +11,13 @@
       </joint>
     </xacro:unless>
+    <!-- for simulation -->
+    <link name="world" />
+    <joint name="robot_to_world" type="fixed">
+      <parent link="world" />
+      <child link="${arm_id}_link0" />
+      <origin xyz="0.0 0.0 0.0" rpy="0.0 0.0 0.0" />
+    </joint>
+    <xacro:property name="joint_damping" value="1.0"/>
+    <!-- end for simulation -->
     <link name="${arm_id}_link0">
       <visual>
@@ -35,4 +44,11 @@
         </geometry>
       </collision>
+      <!-- for simulation -->
+      <inertial>
+        <origin xyz="0 0 0" rpy="0 0 0" />
+        <mass value="3.06" />
+        <inertia ixx="0.3" ixy="0.0" ixz="0.0" iyy="0.3" iyz="0.0" izz="0.3" />
+      </inertial>
+      <!-- end for simulation -->
     </link>
     <link name="${arm_id}_link1">
@@ -60,4 +76,11 @@
         </geometry>
       </collision>
+      <!-- for simulation -->
+      <inertial>
+        <origin xyz="0 0 0" rpy="0 0 0" />
+        <mass value="2.34" />
+        <inertia ixx="0.3" ixy="0.0" ixz="0.0" iyy="0.3" iyz="0.0" izz="0.3" />
+      </inertial>
+      <!-- end for simulation -->
     </link>
     <joint name="${arm_id}_joint1" type="revolute">
@@ -68,4 +91,7 @@
       <axis xyz="0 0 1"/>
       <limit effort="87" lower="-2.8973" upper="2.8973" velocity="2.1750"/>
+      <!-- for simulation -->
+      <dynamics damping="${joint_damping}"/>
+      <!-- end for simulation -->
     </joint>
     <link name="${arm_id}_link2">
@@ -93,4 +119,11 @@
         </geometry>
       </collision>
+      <!-- for simulation -->
+      <inertial>
+        <origin xyz="0 0 0" rpy="0 0 0" />
+        <mass value="2.36" />
+        <inertia ixx="0.3" ixy="0.0" ixz="0.0" iyy="0.3" iyz="0.0" izz="0.3" />
+      </inertial>
+      <!-- end for simulation -->
     </link>
     <joint name="${arm_id}_joint2" type="revolute">
@@ -101,4 +134,7 @@
       <axis xyz="0 0 1"/>
       <limit effort="87" lower="-1.7628" upper="1.7628" velocity="2.1750"/>
+      <!-- for simulation -->
+      <dynamics damping="${joint_damping}"/>
+      <!-- end for simulation -->
     </joint>
     <link name="${arm_id}_link3">
@@ -126,4 +162,11 @@
         </geometry>
       </collision>
+      <!-- for simulation -->
+      <inertial>
+        <origin xyz="0 0 0" rpy="0 0 0" />
+        <mass value="2.38" />
+        <inertia ixx="0.3" ixy="0.0" ixz="0.0" iyy="0.3" iyz="0.0" izz="0.3" />
+      </inertial>
+      <!-- end for simulation -->
     </link>
     <joint name="${arm_id}_joint3" type="revolute">
@@ -134,4 +177,7 @@
       <axis xyz="0 0 1"/>
       <limit effort="87" lower="-2.8973" upper="2.8973" velocity="2.1750"/>
+      <!-- for simulation -->
+      <dynamics damping="${joint_damping}"/>
+      <!-- end for simulation -->
     </joint>
     <link name="${arm_id}_link4">
@@ -159,4 +205,11 @@
         </geometry>
       </collision>
+      <!-- for simulation -->
+      <inertial>
+        <origin xyz="0 0 0" rpy="0 0 0" />
+        <mass value="2.43" />
+        <inertia ixx="0.3" ixy="0.0" ixz="0.0" iyy="0.3" iyz="0.0" izz="0.3" />
+      </inertial>
+      <!-- end for simulation -->
     </link>
     <joint name="${arm_id}_joint4" type="revolute">
@@ -167,4 +220,7 @@
       <axis xyz="0 0 1"/>
       <limit effort="87" lower="-3.0718" upper="-0.0698" velocity="2.1750"/>
+      <!-- for simulation -->
+      <dynamics damping="${joint_damping}"/>
+      <!-- end for simulation -->
     </joint>
     <link name="${arm_id}_link5">
@@ -210,4 +266,11 @@
         </geometry>
       </collision>
+      <!-- for simulation -->
+      <inertial>
+        <origin xyz="0 0 0" rpy="0 0 0" />
+        <mass value="3.5" />
+        <inertia ixx="0.3" ixy="0.0" ixz="0.0" iyy="0.3" iyz="0.0" izz="0.3" />
+      </inertial>
+      <!-- end for simulation -->
     </link>
     <joint name="${arm_id}_joint5" type="revolute">
@@ -218,4 +281,7 @@
       <axis xyz="0 0 1"/>
       <limit effort="12" lower="-2.8973" upper="2.8973" velocity="2.6100"/>
+      <!-- for simulation -->
+      <dynamics damping="${joint_damping}"/>
+      <!-- end for simulation -->
     </joint>
     <link name="${arm_id}_link6">
@@ -243,4 +309,11 @@
         </geometry>
       </collision>
+      <!-- for simulation -->
+      <inertial>
+        <origin xyz="0 0 0" rpy="0 0 0" />
+        <mass value="1.47" />
+        <inertia ixx="0.3" ixy="0.0" ixz="0.0" iyy="0.3" iyz="0.0" izz="0.3" />
+      </inertial>
+      <!-- end for simulation -->
     </link>
     <joint name="${arm_id}_joint6" type="revolute">
@@ -251,4 +324,7 @@
       <axis xyz="0 0 1"/>
       <limit effort="12" lower="-0.0175" upper="3.7525" velocity="2.6100"/>
+      <!-- for simulation -->
+      <dynamics damping="${joint_damping}"/>
+      <!-- end for simulation -->
     </joint>
     <link name="${arm_id}_link7">
@@ -276,4 +352,11 @@
         </geometry>
       </collision>
+      <!-- for simulation -->
+      <inertial>
+        <origin xyz="0 0 0" rpy="0 0 0" />
+        <mass value="0.45" />
+        <inertia ixx="0.3" ixy="0.0" ixz="0.0" iyy="0.3" iyz="0.0" izz="0.3" />
+      </inertial>
+       <!-- end for simulation -->
     </link>
     <joint name="${arm_id}_joint7" type="revolute">
@@ -284,4 +367,7 @@
       <axis xyz="0 0 1"/>
       <limit effort="12" lower="-2.8973" upper="2.8973" velocity="2.6100"/>
+      <!-- for simulation -->
+      <dynamics damping="${joint_damping}"/>
+      <!-- end for simulation -->
     </joint>
     <link name="${arm_id}_link8">
@@ -304,4 +390,11 @@
         </geometry>
       </collision>
+      <!-- for simulation -->
+      <inertial>
+        <origin xyz="0 0 0" rpy="0 0 0" />
+        <mass value="0.0" />
+        <inertia ixx="0.3" ixy="0.0" ixz="0.0" iyy="0.3" iyz="0.0" izz="0.3" />
+      </inertial>
+      <!-- end for simulation -->
     </link>
     <joint name="${arm_id}_joint8" type="fixed">

File: franka_description/robots/panda_arm_hand.urdf.xacro (robot description, xacro)
@@ -3,4 +3,13 @@
   <xacro:include filename="$(find franka_description)/robots/panda_arm.xacro"/>
   <xacro:include filename="$(find franka_description)/robots/hand.xacro"/>
+  <!-- for simulation -->
+  <xacro:include filename="$(find franka_description)/robots/panda.gazebo.xacro"/>
+  <xacro:include filename="panda.transmission.xacro"/>
+  <!-- end for simulation -->
+  <!-- for simulation -->
+  <xacro:arg name="robot_name" default="panda"/>
+  <xacro:panda_gazebo robot_name="$(arg robot_name)" />
+  <xacro:panda_transmission robot_name="$(arg robot_name)" load_hand="true" />
+  <!-- end for simulation -->
   <xacro:panda_arm safety_distance="0.03"/>
   <xacro:hand ns="panda" rpy="0 0 ${-pi/4}" connected_to="panda_link8" safety_distance="0.03"/>
