Commit message: (1) Modified Panda_arm xacro to be connect-able to other robots irrespective of world link and (2) added an automatically generated panda_arm_hand URDF using rosrun xacro conversion. This urdf is needed for PyBullet use of pure franka.

File: franka_description/robots/panda_arm.xacro (robot description, xacro)
@@ -2,4 +2,8 @@
 <robot xmlns:xacro="http://www.ros.org/wiki/xacro" name="panda">
   <xacro:macro name="panda_arm" params="arm_id:='panda' description_pkg:='franka_description' connected_to:='' xyz:='0 0 0' rpy:='0 0 0'">
+    <!--
+    Panda is either connected to an external link
+    or to a virtual world link.
+    -->
     <xacro:unless value="${not connected_to}">
       <joint name="${arm_id}_joint_${connected_to}" type="fixed">
@@ -10,10 +14,12 @@
     </xacro:unless>
     <!-- for simulation -->
-    <link name="world" />
-    <joint name="robot_to_world" type="fixed">
-      <parent link="world" />
-      <child link="${arm_id}_link0" />
-      <origin xyz="0.0 0.0 0.0" rpy="0.0 0.0 0.0" />
-    </joint>
+    <xacro:if value="${not connected_to}">
+      <link name="world" />
+      <joint name="robot_to_world" type="fixed">
+        <parent link="world" />
+        <child link="${arm_id}_link0" />
+        <origin xyz="0.0 0.0 0.0" rpy="0.0 0.0 0.0" />
+      </joint>
+      </xacro:if>
     <xacro:property name="joint_damping" value="1.0"/>
     <!-- end for simulation -->
