Commit message: trying to fix simulation

File: franka_description/robots/panda.gazebo.xacro (robot description, xacro)
@@ -1,77 +1,31 @@
-<?xml version="1.0"?>
+<?xml version='1.0' encoding='utf-8'?>
 <robot xmlns:xacro="http://www.ros.org/wiki/xacro">
-    <xacro:macro name="panda_gazebo" params="robot_name">
-        <!-- Link0 -->
-        <gazebo reference="${robot_name}_link0">
-            <material>Gazebo/Grey</material>
-            <mu1>0.2</mu1>
-            <mu2>0.2</mu2>
-        </gazebo>
-        <!-- Link1 -->
-        <gazebo reference="${robot_name}_link1">
-            <material>Gazebo/White</material>
-            <mu1>0.2</mu1>
-            <mu2>0.2</mu2>
-        </gazebo>
-        <!-- Link2 -->
-        <gazebo reference="${robot_name}_link2">
-            <material>Gazebo/White</material>
-            <mu1>0.2</mu1>
-            <mu2>0.2</mu2>
-        </gazebo>
-        <!-- Link3 -->
-        <gazebo reference="${robot_name}_link3">
-            <material>Gazebo/White</material>
-            <mu1>0.2</mu1>
-            <mu2>0.2</mu2>
-        </gazebo>
-        <!-- Link4 -->
-        <gazebo reference="${robot_name}_link4">
-            <material>Gazebo/White</material>
-            <mu1>0.2</mu1>
-            <mu2>0.2</mu2>
-        </gazebo>
-        <!-- Link5 -->
-        <gazebo reference="${robot_name}_link5">
-            <material>Gazebo/White</material>
-            <mu1>0.2</mu1>
-            <mu2>0.2</mu2>
-        </gazebo>
-        <!-- Link6 -->
-        <gazebo reference="${robot_name}_link6">
-            <material>Gazebo/White</material>
-            <mu1>0.2</mu1>
-            <mu2>0.2</mu2>
-        </gazebo>
-        <!-- Link7 -->
-        <gazebo reference="${robot_name}_link7">
-            <material>Gazebo/Grey</material>
-            <mu1>0.2</mu1>
-            <mu2>0.2</mu2>
-        </gazebo>
-        <!-- Link8 -->
-        <gazebo reference="${robot_name}_link8">
-            <material>Gazebo/Grey</material>
-            <mu1>0.2</mu1>
-            <mu2>0.2</mu2>
-        </gazebo>
-        <!-- LinkHand -->
-        <gazebo reference="${robot_name}_hand">
-            <material>Gazebo/Grey</material>
-            <mu1>0.2</mu1>
-            <mu2>0.2</mu2>
-        </gazebo>
-        <!-- LinkRightFinger -->
-        <gazebo reference="${robot_name}_rightfinger">
-            <material>Gazebo/Grey</material>
-            <mu1>0.2</mu1>
-            <mu2>0.2</mu2>
-        </gazebo>
-        <!-- LinkLeftFinger -->
-        <gazebo reference="${robot_name}_leftfinger">
-            <material>Gazebo/Grey</material>
-            <mu1>0.2</mu1>
-            <mu2>0.2</mu2>
-        </gazebo>
+    <xacro:macro name="panda_gazebo" params="arm_id">
+        <xacro:macro name="arm_gazebo" params="link">
+            <gazebo reference="${link}">
+                <material>Gazebo/White</material>
+                <mu1>0.2</mu1>
+                <mu2>0.2</mu2>
+            </gazebo>
+        </xacro:macro>
+        <xacro:macro name="hand_gazebo" params="link">
+            <gazebo reference="${link}">
+                <material>Gazebo/Grey</material>
+                <mu1>0.2</mu1>
+                <mu2>0.2</mu2>
+            </gazebo>
+        </xacro:macro>
+        <xacro:arm_gazebo link="${arm_id}_link0"/>
+        <xacro:arm_gazebo link="${arm_id}_link1"/>
+        <xacro:arm_gazebo link="${arm_id}_link2"/>
+        <xacro:arm_gazebo link="${arm_id}_link3"/>
+        <xacro:arm_gazebo link="${arm_id}_link4"/>
+        <xacro:arm_gazebo link="${arm_id}_link5"/>
+        <xacro:arm_gazebo link="${arm_id}_link6"/>
+        <xacro:hand_gazebo link="${arm_id}_link7"/>
+        <xacro:hand_gazebo link="${arm_id}_link8"/>
+        <xacro:hand_gazebo link="${arm_id}_hand"/>
+        <xacro:hand_gazebo link="${arm_id}_rightfinger"/>
+        <xacro:hand_gazebo link="${arm_id}_leftfinger"/>
     </xacro:macro>
 </robot>

File: franka_description/robots/panda.transmission.xacro (robot description, xacro)
@@ -5,5 +5,7 @@
         <gazebo>
             <plugin name="gazebo_ros_control" filename="libgazebo_ros_control.so">
-                <!-- <robotNamespace>/${robot_name}</robotNamespace> -->
+                <robotSimType>gazebo_ros_control/DefaultRobotHWSim</robotSimType>
+                <legacyModeNS>true</legacyModeNS>
+                <robotNamespace>/robot</robotNamespace>
             </plugin>
         </gazebo>

File: franka_description/robots/panda_arm_hand.urdf.xacro (robot description, xacro)
@@ -5,12 +5,12 @@
   <!-- for simulation -->
   <xacro:include filename="$(find franka_description)/robots/panda.gazebo.xacro"/>
-  <xacro:include filename="panda.transmission.xacro"/>
+  <xacro:include filename="$(find franka_description)/robots/panda.control.xacro"/>
   <!-- end for simulation -->
   <xacro:panda_arm />
   <xacro:hand ns="panda" rpy="0 0 ${-pi/4}" connected_to="panda_link8"/>
+  <xacro:panda_gazebo arm_id="panda"/>
+  <xacro:panda_control arm_id="panda" load_hand="true" />
   <!-- for simulation -->
   <xacro:arg name="robot_name" default="panda"/>
-  <xacro:panda_gazebo robot_name="$(arg robot_name)" />
-  <xacro:panda_transmission robot_name="$(arg robot_name)" load_hand="true" />
   <!-- end for simulation -->
 </robot>
